Commit message: Updating the my_world.xacro file for Robot Enhancement

File: catkin_ws/src/my_robot/urdf/my_robot.xacro (robot description, xacro)
@@ -55,3 +55,77 @@
     </visual>
   </link>
+<!-- Left Wheel -->
+  <link name='left_wheel'>
+    <pose>0 0 0 0 0 0</pose>
+    <inertial>
+      <mass value = "5"/>
+      <origin xyz="0 0 0" rpy=" 0 1.5707 1.5707"/>
+      <inertia
+        ixx="0.1" ixy="0" ixz="0"
+        iyy="0.1" iyz="0"
+        izz="0.1"
+      />
+    </inertial>
+    <collision name='collision'>
+      <origin xyz="0 0 0" rpy=" 0 1.5707 1.5707"/>
+      <geometry>
+        <!-- <cylinder>
+          <radius>0.1</radius>
+          <length>0.05</length>
+       </cylinder> -->
+       <cylinder radius="0.1" length="0.05"/>
+      </geometry>
+    </collision>
+    <visual>
+      <origin xyz="0 0 0" rpy=" 0 1.5707 1.5707"/>
+      <geometry>
+        <!-- <cylinder>
+          <radius>0.1</radius>
+          <length>0.05</length>
+       </cylinder> -->
+       <cylinder radius="0.1" length="0.05"/>
+      </geometry>
+    </visual>
+  </link>
+  <joint type="continuous" name="left_wheel_hinge">
+    <origin xyz="0 0.15 0" rpy="0 0 0"/>
+    <child link="left_wheel"/>
+    <parent link="chassis"/>
+    <axis xyz="0 1 0" rpy="0 0 0"/>
+    <limit effort="10000" velocity="1000"/>
+    <dynamics damping="1.0" friction="1.0"/>
+  </joint>
+<!-- Right Wheel -->
+  <link name='right_wheel'>
+    <pose>0 0 0 0 0 0</pose>
+    <inertial>
+      <mass value = "5"/>
+      <origin xyz="0 0 0" rpy=" 0 1.5707 1.5707"/>
+      <inertia
+        ixx="0.1" ixy="0" ixz="0"
+        iyy="0.1" iyz="0"
+        izz="0.1"
+      />
+    </inertial>
+    <collision name='collision'>
+      <origin xyz="0 0 0" rpy=" 0 1.5707 1.5707"/>
+      <geometry>
+       <cylinder radius="0.1" length="0.05"/>
+      </geometry>
+    </collision>
+    <visual>
+      <origin xyz="0 0 0" rpy=" 0 1.5707 1.5707"/>
+      <geometry>
+       <cylinder radius="0.1" length="0.05"/>
+      </geometry>
+    </visual>
+  </link>
+  <joint type="continuous" name="right_wheel_hinge">
+    <origin xyz="0 -0.15 0" rpy="0 0 0"/>
+    <child link="right_wheel"/>
+    <parent link="chassis"/>
+    <axis xyz="0 1 0" rpy="0 0 0"/>
+    <limit effort="10000" velocity="1000"/>
+    <dynamics damping="1.0" friction="1.0"/>
+  </joint>
 </robot>

Commit message: Updating my_robot.xacro file to add a camera

File: catkin_ws/src/my_robot/urdf/my_robot.xacro (robot description, xacro)
@@ -55,5 +55,5 @@
     </visual>
   </link>
-<!-- Left Wheel -->
+<!-- adding Left Wheel -->
   <link name='left_wheel'>
     <pose>0 0 0 0 0 0</pose>
@@ -96,5 +96,5 @@
     <dynamics damping="1.0" friction="1.0"/>
   </joint>
-<!-- Right Wheel -->
+<!-- adding Right Wheel -->
   <link name='right_wheel'>
     <pose>0 0 0 0 0 0</pose>
@@ -129,3 +129,34 @@
     <dynamics damping="1.0" friction="1.0"/>
   </joint>
+<!-- adding a Camera -->
+   <link name = 'camera'>
+    <pose>0 0 0 0 0 0</pose>
+    <inertial>
+        <mass value="0.1"/>
+        <origin xyz = "0 0 0" rpy=" 0 0 0"/>
+        <inertia
+            ixx="1e-6" ixy="0" ixz="0"
+            iyy="1e-6" iyz="0"
+            izz="1e-6"
+        />
+    </inertial>
+    <collision name='collision'>
+        <origin xyz = "0 0 0" rpy=" 0 0 0"/>
+        <geometry>
+            <box size = "0.05 0.05 0.05"/>
+        </geometry>
+    </collision>
+    <visual>
+        <origin xyz = "0 0 0" rpy=" 0 0 0"/>
+        <geometry>
+            <box size = "0.05 0.05 0.05"/>
+        </geometry>
+    </visual>
+   </link>
+   <joint type="fixed" name="camera_joint">
+    <origin xyz="0.2 0 0" rpy="0 0 0"/>
+    <child link="camera"/>
+    <parent link="chassis"/>
+    <axis xyz="0 1 0"/>
+   </joint>
 </robot>

Commit message: Adding the 'link' and 'joint' tag for "hokuyo" sensor in .xacro file

File: catkin_ws/src/my_robot/urdf/my_robot.xacro (robot description, xacro)
@@ -67,5 +67,5 @@
       />
     </inertial>
-    <collision name='collision'>
+    <collision name='left_wheel_collision'>
       <origin xyz="0 0 0" rpy=" 0 1.5707 1.5707"/>
       <geometry>
@@ -77,5 +77,5 @@
       </geometry>
     </collision>
-    <visual>
+    <visual name='left_wheel_visual'>
       <origin xyz="0 0 0" rpy=" 0 1.5707 1.5707"/>
       <geometry>
@@ -108,5 +108,5 @@
       />
     </inertial>
-    <collision name='collision'>
+    <collision name='right_wheel_collision'>
       <origin xyz="0 0 0" rpy=" 0 1.5707 1.5707"/>
       <geometry>
@@ -114,5 +114,5 @@
       </geometry>
     </collision>
-    <visual>
+    <visual name='right_wheel_visual'>
       <origin xyz="0 0 0" rpy=" 0 1.5707 1.5707"/>
       <geometry>
@@ -141,5 +141,5 @@
         />
     </inertial>
-    <collision name='collision'>
+    <collision name='camera_collision'>
         <origin xyz = "0 0 0" rpy=" 0 0 0"/>
         <geometry>
@@ -147,5 +147,5 @@
         </geometry>
     </collision>
-    <visual>
+    <visual name='camera_visual'>
         <origin xyz = "0 0 0" rpy=" 0 0 0"/>
         <geometry>
@@ -155,8 +155,38 @@
    </link>
    <joint type="fixed" name="camera_joint">
-    <origin xyz="0.2 0 0" rpy="0 0 0"/>
-    <child link="camera"/>
-    <parent link="chassis"/>
-    <axis xyz="0 1 0"/>
+        <origin xyz="0.2 0 0" rpy="0 0 0"/>
+        <parent link="chassis"/>
+        <child link="camera"/>
+        <axis xyz="0 1 0"/>
    </joint>
+<!-- adding Hokuyo sensor -->
+    <link name = 'hokuyo'>
+        <inertial>
+            <mass value ="1e-5"/>
+            <origin xyz="0 0 0" rpy="0 0 0"/>
+            <inertia
+                ixx="1e-6" ixy="0" ixz="0"
+                iyy="1e-6" iyz="0"
+                izz="1e-6"
+            />
+        </inertial>
+        <collision name='hokuyo_collision'>
+            <origin xyz = "0 0 0" rpy="0 0 0"/>
+            <geometry>
+                <box size = "0.1 0.1 0.1"/>
+            </geometry>
+        </collision>
+        <visual name='hokuyo_visual'>
+            <origin xyz = "0 0 0" rpy="0 0 0"/>
+            <geometry>
+                <mesh filename="package://my_robot/meshes/hokuyo.dae"/>
+            </geometry>
+        </visual>
+    </link>
+	  <joint type="fixed" name="hokuyo_joint">
+        <origin xyz="0.15 0 0.1" rpy="0 0 0"/>
+        <parent link="chassis"/>
+        <child link="hokuyo"/>
+        <axis xyz = "0 1 0"/>
+    </joint>
 </robot>

Commit message: Updating the color of wheels, chassis of a robot and that of a camera.
Add the 'material' tags in the urdf/my_robot.xcro file

Use link_names as a reference

File: catkin_ws/src/my_robot/urdf/my_robot.xacro (robot description, xacro)
@@ -7,4 +7,5 @@
     <child link="chassis" />
   </joint>
+<!-- for main Chassis -->
   <link name='chassis'>
     <pose>0 0 0.1 0 0 0</pose>
@@ -184,5 +185,5 @@
         </visual>
     </link>
-	  <joint type="fixed" name="hokuyo_joint">
+    <joint type="fixed" name="hokuyo_joint">
         <origin xyz="0.15 0 0.1" rpy="0 0 0"/>
         <parent link="chassis"/>
@@ -190,3 +191,19 @@
         <axis xyz = "0 1 0"/>
     </joint>
+<!-- Changing the color of Left Wheel -->
+<gazebo reference="left_wheel">
+  <material>Gazebo/Black</material>
+</gazebo>
+<!-- Changing the color of Right Wheel -->
+<gazebo reference="right_wheel">
+  <material>Gazebo/Black</material>
+</gazebo>
+<!-- Changing the color of Chassis -->
+<gazebo reference="chassis">
+  <material>Gazebo/Red</material>
+</gazebo>
+<!-- Changing the color of Camera -->
+<gazebo reference="camera">
+  <material>Gazebo/Blue</material>
+</gazebo>
 </robot>

Commit message: Updating urdf/my_robot.xacro file & adding my_world.urdf file.
1. Adjusted spaces in the urdf/my_robot.xacro file
2. Added my_world.urdf file. This file provides the plugins for
   camera sensor, Hokuyo sensor, and wheel joints.

File: catkin_ws/src/my_robot/urdf/my_robot.xacro (robot description, xacro)
@@ -192,18 +192,18 @@
     </joint>
 <!-- Changing the color of Left Wheel -->
-<gazebo reference="left_wheel">
-  <material>Gazebo/Black</material>
-</gazebo>
+    <gazebo reference="left_wheel">
+      <material>Gazebo/Black</material>
+    </gazebo>
 <!-- Changing the color of Right Wheel -->
-<gazebo reference="right_wheel">
-  <material>Gazebo/Black</material>
-</gazebo>
+    <gazebo reference="right_wheel">
+      <material>Gazebo/Black</material>
+    </gazebo>
 <!-- Changing the color of Chassis -->
-<gazebo reference="chassis">
-  <material>Gazebo/Red</material>
-</gazebo>
+    <gazebo reference="chassis">
+      <material>Gazebo/Red</material>
+    </gazebo>
 <!-- Changing the color of Camera -->
-<gazebo reference="camera">
-  <material>Gazebo/Blue</material>
-</gazebo>
+    <gazebo reference="camera">
+      <material>Gazebo/Blue</material>
+    </gazebo>
 </robot>

Commit message: Added 'optical' camera link in my_robot.xacro file
01. Did this for getting D of RGB-D sensor:
	Added extra link 'camera_optial_link'
	Added extra joint 'camera_optical_joint'

File: catkin_ws/src/my_robot/urdf/my_robot.xacro (robot description, xacro)
@@ -162,4 +162,12 @@
         <axis xyz="0 1 0"/>
    </joint>
+<!-- 'optical' camera link | for RGB-D camera -->
+  <joint name="camera_optical_joint" type="fixed">
+    <origin xyz="0 0 0" rpy="-1.5707 0 -1.5707"/>
+    <parent link="camera"/>
+    <child link="camera_link_optical"/>
+  </joint>
+  <link name="camera_link_optical">
+  </link>
 <!-- adding Hokuyo sensor -->
     <link name = 'hokuyo'>

Commit message: Updated the parent link name in 'camera_optical_joint'.

File: catkin_ws/src/my_robot/urdf/my_robot.xacro (robot description, xacro)
@@ -165,5 +165,5 @@
   <joint name="camera_optical_joint" type="fixed">
     <origin xyz="0 0 0" rpy="-1.5707 0 -1.5707"/>
-    <parent link="camera"/>
+    <parent link="camera_link"/>
     <child link="camera_link_optical"/>
   </joint>

Commit message: Corrected camera link names in my_robot.xacro
Did this by replacing link names: 'camera' with 'camera_link'

File: catkin_ws/src/my_robot/urdf/my_robot.xacro (robot description, xacro)
@@ -132,5 +132,5 @@
   </joint>
 <!-- adding a Camera -->
-   <link name = 'camera'>
+   <link name = 'camera_link'>
     <pose>0 0 0 0 0 0</pose>
     <inertial>
@@ -159,5 +159,5 @@
         <origin xyz="0.2 0 0" rpy="0 0 0"/>
         <parent link="chassis"/>
-        <child link="camera"/>
+        <child link="camera_link"/>
         <axis xyz="0 1 0"/>
    </joint>
@@ -213,5 +213,5 @@
     </gazebo>
 <!-- Changing the color of Camera -->
-    <gazebo reference="camera">
+    <gazebo reference="camera_link">
       <material>Gazebo/Blue</material>
     </gazebo>
